File: Hardware/KiCad/ADAS_Camera_Emulator/power.kicad_sch (KiCad schematic)
At the start: 0 parts

Commit message: just shematic stuff
Parts:
- added D1: LED_Reg_3.3V, symbol Device:LED_Small
- added D2: LED_Reg_5V, symbol Device:LED_Small
- added D3: LED_12V, symbol Device:LED_Small
- added J2: connector, symbol Connector:Screw_Terminal_01x02
- added R1: 1k6, symbol Device:R_Small
- added R8: 3k8, symbol Device:R_Small
- added R9: 5k5, symbol Device:R_Small
- added S1: 1101M2S3AV2BE2, SWITCH:1000-SERIES_SPDT_, symbol 1101M2S3AV2BE2:1101M2S3AV2BE2
- added TP1: TestPoint_5V, symbol Connector:TestPoint
- added TP2: TestPoint_3.3V, symbol Connector:TestPoint
Connections:
- new net: D2.2 (A), R8.2
- new net: D1.2 (A), R1.2
- new net: D3.2 (A), R9.2
- new net: J2.2 (Pin_2), S1.2
- new net +12V: R9.1, S1.1
- new net +3.3V: R1.1, TP2.1
- new net +5V: R8.1, TP1.1
- new net GND: D1.1 (K), D2.1 (K), D3.1 (K), J2.1 (Pin_1)
- no-connect marks 0 -> 1
Other:
- added sheet BUCK 3.3V (buck3v3.kicad_sch)
- added sheet BUCK 5V (buck5v.kicad_sch)
