File: Hardware/KiCad/ADAS_Camera_Emulator/input_output.kicad_sch (KiCad schematic)
At the start: 0 parts

Commit message: just shematic stuff
Parts:
- added J1: 1747981-1, Library:17479811, symbol 1747981-1:1747981-1
Connections:
- new net +5V: J1.18
- new net CEC: J1.13
- new net DDC Clock: J1.15
- new net DDC Data: J1.16
- new net GND: J1.17, J1.20 (MH1), J1.21 (MH2), J1.22 (MH3), J1.23 (MH4)
- new net Hot Plug Detect: J1.19
- new net TDMS Clock Shield: J1.11
- new net TDMS Clock+: J1.10
- new net TDMS Clock-: J1.12
- new net TDMS Data 0 Shield: J1.8
- new net TDMS Data 0+: J1.7
- new net TDMS Data 0-: J1.9
- new net TDMS Data 1 Shield: J1.5
- new net TDMS Data 1+: J1.4
- new net TDMS Data 1-: J1.6
- new net TDMS Data 2 Shield: J1.2
- new net TDMS Data 2+: J1.1
- new net TDMS Data 2-: J1.3
- no-connect marks 0 -> 1

Commit message: just trying stuff and trying to choose the best materials for the job
Parts:
- added C15, C16: 22p, symbol Device:C_Small
- added D4: LED_Small, symbol Device:LED_Small
- added IC2: TC358743XBG, Toshiba_TC358743XBG:BGA64C65P8X8_600X600X120, symbol TC358743XBG:TC358743XBG
- added IC3: DS90UB953TRHBTQ1, QFN50P500X500X100-33N-D, symbol DS90UB953TRHBTQ1:DS90UB953TRHBTQ1
- added Q1, Q2: BSS123, Package_TO_SOT_SMD:SOT-23, symbol Transistor_FET:BSS123
- added R12, R13: 220R, symbol Device:R_Small
- added R14: 100k, symbol Device:R_Small
- added R15, R16: 4k7, symbol Device:R_Small
- added U2: ADV7611, Package_QFP:LQFP-64-1EP_10x10mm_P0.5mm_EP5x5mm, symbol Interface_HDMI:ADV7611
- added U3: TPD4E02B04DQA, Package_SON:USON-10_2.5x1.0mm_P0.5mm, symbol Power_Protection:TPD4E02B04DQA
- added Y1: 27MHz, symbol Device:Crystal
Connections:
- net +5V: now also Q2.1 (G), R12.1; no longer J1.18
- net CEC: now also U2.61 (CEC)
- net GND: now also Q1.2 (S), Q2.2 (S), U2.65 (GND), U3.3 (G), U3.8 (G)
- net Hot Plug Detect: now also Q1.1 (G), Q2.3 (D), R13.1, R14.2, U2.1 (HPA_A/INT2)
- net TDMS Clock Shield: now also U3.5 (IO4)
- net TDMS Clock+: now also U2.4 (RXA_C+)
- net TDMS Clock-: now also U2.3 (RXA_C-)
- net TDMS Data 0 Shield: now also U3.4 (IO3)
- net TDMS Data 0+: now also U2.7 (RXA_0+)
- net TDMS Data 0-: now also U2.6 (RXA_0-)
- net TDMS Data 1 Shield: now also U3.2 (IO2)
- net TDMS Data 1+: now also U2.10 (RXA_1+)
- net TDMS Data 1-: now also U2.9 (RXA_1-)
- net TDMS Data 2 Shield: now also U3.1 (IO1)
- net TDMS Data 2+: now also U2.13 (RXA_2+)
- net TDMS Data 2-: now also U2.12 (RXA_2-)
- net DDC Clock renamed DDCA_SCL
- net DDCA_SCL: now also R15.2, U2.62 (DDCA_SCL)
- net DDC Data renamed DDCA_SDA
- net DDCA_SDA: now also R16.2, U2.63 (DDCA_SDA)
- new net: C16.2, U2.59 (XTALN), Y1.1
- new net: C15.2, U2.58 (XTALP), Y1.2
- new net: D4.2 (A), R12.2
- new net: D4.1 (K), Q1.3 (D)
- new net HDMI_A_5V: J1.18, R13.2, R14.1, R15.1, R16.1
Other:
- moved on the sheet: J1
