File: Hardware/KiCad/ADAS_Camera_Emulator/interface.kicad_sch (KiCad schematic)
At the start: 0 parts

Commit message: just trying stuff and trying to choose the best materials for the job
Parts:
- added D803: LED_status, LED_SMD:LED_0603_1608Metric, symbol Device:LED_Small
- added J3: Conn_ST_STDC14, symbol Connector:Conn_ST_STDC14
- added R11: 1k6, symbol Device:R_Small
- added SW2: reset, Button_Switch_SMD:SW_Push_1P1T_NO_E-Switch_TL3301NxxxxxG, symbol Switch:SW_Push
Connections:
- new net: D803.2 (A), R11.2
- new net +3.3V: J3.3 (VCC)
- new net GND: D803.1 (K), J3.11 (GNDDetect), J3.5 (GND), J3.7 (GND), SW2.1
- new net LED_status: R11.1
- new net NRST: J3.12 (~{RST}), SW2.2
- new net SWCLK: J3.6 (JCLK/SWCLK)
- new net SWDIO: J3.4 (JTMS/SWDIO)
- new net SWO: J3.8 (JTDO/SWO)
- new net VCP_RX: J3.13 (VCP_RX)
- new net VCP_TX: J3.14 (VCP_TX)
Other:
- note added: "Buttons"
- note added: "LED indicator"
- note added: "ST LINK / SWD Connector"
